Commit message: update urdf

File: src/vacumm_description/urdf/vacumm.xacro (robot description, xacro)
@@ -29,7 +29,7 @@
         <pose>0 0.1 0 0 0</pose>
         <visual name="chassis">
-            <origin xyz="0 0 0.2" rpy="0 0 0" />
+            <origin xyz="0 0 0.15" rpy="0 0 0" />
             <geometry>
-                <cylinder radius="0.1" length="0.4"/>
+                <cylinder radius="0.1" length="0.3"/>
             </geometry>
             <material name="green" />

Commit message: update urdf

File: src/vacumm_description/urdf/vacumm.xacro (robot description, xacro)
@@ -28,4 +28,14 @@
     <link name="link_base">
         <pose>0 0.1 0 0 0</pose>
+        <inertial>
+            <mass value="5"/>
+            <origin rpy="0 0 0" xyz="0 0 0.1"/>
+            <inertia ixx="0.0395416666667" ixy="0" ixz="0" iyy="0.106208333333" iyz="0" izz="0.106208333333"/>
+        </inertial>
+        <collision name="collision_chassis">
+        <geometry>
+            <cylinder radius="0.1" length="0.3"/>
+        </geometry>
+        </collision>
         <visual name="chassis">
             <origin xyz="0 0 0.15" rpy="0 0 0" />
@@ -49,4 +59,15 @@
     </link>
     <link name="link_left_wheel">
+        <inertial>
+            <mass value="0.2"/>
+            <origin rpy="0 1.5707 1.5707" xyz="0 0 0"/>
+            <inertia ixx="0.000526666666667" ixy="0" ixz="0" iyy="0.000526666666667" iyz="0" izz="0.001"/>
+        </inertial>
+        <collision name="link_left_wheel_collision">
+            <origin rpy="0 1.5707 1.5707" xyz="0 0 0"/>
+            <geometry>
+                <cylinder length="0.04" radius="0.1"/>
+            </geometry>
+        </collision>
         <visual name="left_wheel" >
             <origin xyz="0 0 0" rpy="0 1.5707 1.5707" />
@@ -57,4 +78,15 @@
     </link>
     <link name="link_right_wheel">
+        <inertial>
+            <mass value="0.2"/>
+            <origin rpy="0 1.5707 1.5707" xyz="0 0 0"/>
+            <inertia ixx="0.000526666666667" ixy="0" ixz="0" iyy="0.000526666666667" iyz="0" izz="0.001"/>
+        </inertial>
+        <collision name="link_right_wheel_collision">
+            <origin rpy="0 1.5707 1.5707" xyz="0 0 0"/>
+            <geometry>
+                <cylinder length="0.04" radius="0.1"/>
+            </geometry>
+        </collision>
         <visual name="right_wheel" >
             <origin xyz="0 0 0" rpy="0 1.5707 1.5707" />

Commit message: update urdf

File: src/vacumm_description/urdf/vacumm.xacro (robot description, xacro)
@@ -5,36 +5,41 @@
     </material>
     <gazebo reference="link_base">
+        <material>Gazebo/White</material>
+        <turnGravityOff>false</turnGravityOff>
     </gazebo>
     <gazebo reference="link_left_Wheel">
+        <mu1 value="1.0"/>
+        <mu2 value="1.0"/>
+        <kp value="10000000.0"/>
+        <kd value="1.0"/>
+        <fdir1 value="1 0 0"/>
+        <material>Gazebo/Grey</material>
+        <turnGravityOff>false</turnGravityOff>
     </gazebo>
     <gazebo reference="link_right_wheel">
+        <mu1 value="1.0"/>
+        <mu2 value="1.0"/>
+        <kp value="10000000.0"/>
+        <kd value="1.0"/>
+        <fdir1 value="1 0 0"/>
+        <material>Gazebo/Grey</material>
+        <turnGravityOff>false</turnGravityOff>
     </gazebo>
     <gazebo>
-    <plugin filename="libgazebo_ros_diff_drive.so" name="differential_drive_controller">
-      <legacyMode>false</legacyMode>
-      <alwaysOn>true</alwaysOn>
-      <updateRate>20</updateRate>
-      <leftJoint>joint_left_wheel</leftJoint>
-      <rightJoint>joint_right_wheel</rightJoint>
-      <wheelSeparation>0.235</wheelSeparation>
-      <wheelDiameter>0.08</wheelDiameter>
-      <torque>0.1</torque>
-      <commandTopic>cmd_vel</commandTopic>
-      <odometryTopic>odom</odometryTopic>
-      <odometryFrame>odom</odometryFrame>
-      <robotBaseFrame>link_base</robotBaseFrame>
-    </plugin>
-  </gazebo>
+        <plugin name="gazebo_ros_control" filename="libgazebo_ros_control.so">
+            <legacyMode>false</legacyMode>
+        </plugin>
+    </gazebo>
     <link name="link_base">
         <pose>0 0.1 0 0 0</pose>
         <inertial>
-            <mass value="5"/>
+            <mass value="2"/>
             <origin rpy="0 0 0" xyz="0 0 0.1"/>
             <inertia ixx="0.0395416666667" ixy="0" ixz="0" iyy="0.106208333333" iyz="0" izz="0.106208333333"/>
         </inertial>
         <collision name="collision_chassis">
-        <geometry>
-            <cylinder radius="0.1" length="0.3"/>
-        </geometry>
+            <geometry>
+                <cylinder radius="0.1" length="0.3"/>
+            </geometry>
         </collision>
         <visual name="chassis">
@@ -96,19 +101,39 @@
         </visual>
     </link>
-    <joint name="joint_left_wheel" type="continuous">
+    <joint name="left_wheel_joint" type="continuous">
         <parent link="link_base"/>
         <child link="link_left_wheel"/>
         <origin xyz="0 0.11 -0.02" rpy="0 0 0"/>
         <axis xyz="0 1 0" rpy="0 0 0"/>
-        <limit effort="10000" velocity="1000"/>
+        <limit effort="0.4" velocity="0.299"/>
         <joint_properties damping="1.0" friction="1.0" />
     </joint>
-    <joint name="joint_right_wheel" type="continuous">
+    <joint name="right_wheel_joint" type="continuous">
         <parent link="link_base"/>
         <child link="link_right_wheel"/>
         <origin xyz="0 -0.11 -0.02" rpy="0 0 0"/>
         <axis xyz="0 1 0" rpy="0 0 0"/>
-        <limit effort="10000" velocity="1000"/>
+        <limit effort="0.4" velocity="0.299"/>
         <joint_properties damping="1.0" friction="1.0" />
     </joint>
+    <transmission name="left_wheel_joint_trans" type="SimpleTransmission">
+        <type>transmission_interface/SimpleTransmission</type>
+        <joint name="left_wheel_joint">
+            <hardwareInterface>hardware_interface/VelocityJointInterface</hardwareInterface>
+        </joint>
+        <actuator name="left_wheel_joint_motor">
+            <hardwareInterface>hardware_interface/VelocityJointInterface</hardwareInterface>
+            <mechanicalReduction>1</mechanicalReduction>
+        </actuator>
+    </transmission>
+    <transmission name="right_wheel_joint_trans" type="SimpleTransmission">
+        <type>transmission_interface/SimpleTransmission</type>
+        <joint name="right_wheel_joint">
+            <hardwareInterface>hardware_interface/VelocityJointInterface</hardwareInterface>
+        </joint>
+        <actuator name="right_wheel_joint_motor">
+            <hardwareInterface>hardware_interface/VelocityJointInterface</hardwareInterface>
+            <mechanicalReduction>1</mechanicalReduction>
+        </actuator>
+    </transmission>
 </robot>

Commit message: update

File: src/vacumm_description/urdf/vacumm.xacro (robot description, xacro)
@@ -11,6 +11,6 @@
         <mu1 value="1.0"/>
         <mu2 value="1.0"/>
-        <kp value="10000000.0"/>
-        <kd value="1.0"/>
+        <kp value="0.5"/>
+        <ki value="2.0"/>
         <fdir1 value="1 0 0"/>
         <material>Gazebo/Grey</material>
@@ -20,6 +20,6 @@
         <mu1 value="1.0"/>
         <mu2 value="1.0"/>
-        <kp value="10000000.0"/>
-        <kd value="1.0"/>
+        <kp value="0.5"/>
+        <ki value="2"/>
         <fdir1 value="1 0 0"/>
         <material>Gazebo/Grey</material>
@@ -39,4 +39,5 @@
         </inertial>
         <collision name="collision_chassis">
+            <origin xyz="0 0 0.15" rpy="0 0 0" />
             <geometry>
                 <cylinder radius="0.1" length="0.3"/>
@@ -72,5 +73,5 @@
             <origin rpy="0 1.5707 1.5707" xyz="0 0 0"/>
             <geometry>
-                <cylinder length="0.04" radius="0.1"/>
+                <cylinder radius="0.04" length="0.01"/>
             </geometry>
         </collision>
@@ -91,5 +92,5 @@
             <origin rpy="0 1.5707 1.5707" xyz="0 0 0"/>
             <geometry>
-                <cylinder length="0.04" radius="0.1"/>
+                <cylinder radius="0.04" length="0.01"/>
             </geometry>
         </collision>

Commit message: update

File: src/vacumm_description/urdf/vacumm.xacro (robot description, xacro)
@@ -1,25 +1,46 @@
 <?xml version="1.0"?>
-<robot name="vacumm_robot" xmlns:xacro="http://www.ros.org/wiki/xacro">
-    <material name="green">
-        <color rgba="0.0 0.8 0.0 1.0"/>
-    </material>
-    <gazebo reference="link_base">
+<robot name="vacumm_robot" xmlns:xacro="https://www.ros.org/wiki/xacro" >
+  <material name="black">
+    <color rgba="0.0 0.0 0.0 1.0"/>
+  </material>
+  <material name="blue">
+    <color rgba="0.203125 0.23828125 0.28515625 1.0"/>
+  </material>
+  <material name="green">
+    <color rgba="0.0 0.8 0.0 1.0"/>
+  </material>
+  <material name="grey">
+    <color rgba="0.2 0.2 0.2 1.0"/>
+  </material>
+  <material name="orange">
+    <color rgba="1.0 0.423529411765 0.0392156862745 1.0"/>
+  </material>
+  <material name="brown">
+    <color rgba="0.870588235294 0.811764705882 0.764705882353 1.0"/>
+  </material>
+  <material name="red">
+    <color rgba="0.80078125 0.12890625 0.1328125 1.0"/>
+  </material>
+  <material name="white">
+    <color rgba="1.0 1.0 1.0 1.0"/>
+  </material>
+  <gazebo reference="base_link">
         <material>Gazebo/White</material>
         <turnGravityOff>false</turnGravityOff>
     </gazebo>
-    <gazebo reference="link_left_Wheel">
+    <gazebo reference="left_Wheel_link">
         <mu1 value="1.0"/>
         <mu2 value="1.0"/>
-        <kp value="0.5"/>
-        <ki value="2.0"/>
+        <kp value="600000"/>
+        <kd value="3"/>
         <fdir1 value="1 0 0"/>
         <material>Gazebo/Grey</material>
         <turnGravityOff>false</turnGravityOff>
     </gazebo>
-    <gazebo reference="link_right_wheel">
+    <gazebo reference="right_wheel_link">
         <mu1 value="1.0"/>
         <mu2 value="1.0"/>
-        <kp value="0.5"/>
-        <ki value="2"/>
+        <kp value="600000"/>
+        <kd value="3"/>
         <fdir1 value="1 0 0"/>
         <material>Gazebo/Grey</material>
@@ -31,92 +52,107 @@
         </plugin>
     </gazebo>
-    <link name="link_base">
-        <pose>0 0.1 0 0 0</pose>
-        <inertial>
-            <mass value="2"/>
-            <origin rpy="0 0 0" xyz="0 0 0.1"/>
-            <inertia ixx="0.0395416666667" ixy="0" ixz="0" iyy="0.106208333333" iyz="0" izz="0.106208333333"/>
-        </inertial>
-        <collision name="collision_chassis">
-            <origin xyz="0 0 0.15" rpy="0 0 0" />
-            <geometry>
-                <cylinder radius="0.1" length="0.3"/>
-            </geometry>
-        </collision>
-        <visual name="chassis">
-            <origin xyz="0 0 0.15" rpy="0 0 0" />
-            <geometry>
-                <cylinder radius="0.1" length="0.3"/>
-            </geometry>
-            <material name="green" />
-        </visual>
-        <visual name="front_castor">
-            <origin xyz="0.065 0 -0.025" rpy="0 0 0" />
-            <geometry>
-                <cylinder radius="0.025" length="0.05"/>
-            </geometry>
-        </visual>
-        <visual name="back_castor" >
-            <origin xyz="-0.065 0 -0.025" rpy="0 0 0" />
-            <geometry>
-                <cylinder radius="0.025" length="0.05"/>
-            </geometry>
-        </visual>
+  <link name="base_link">
+    <!-- pose and inertial -->
+    <pose>0 0 0.1 0 0 0</pose>
+    <inertial>
+      <mass value="5"/>
+      <origin rpy="0 0 0" xyz="0 0 0.1"/>
+      <inertia ixx="0.0395416666667" ixy="0" ixz="0" iyy="0.106208333333" iyz="0" izz="0.106208333333"/>
+    </inertial>
+    <collision name="collision_chassis">
+      <geometry>
+        <box size="0.5 0.3 0.07"/>
+      </geometry>
+    </collision>
+    <visual>
+      <origin rpy="0 0 0" xyz="0 0 0"/>
+      <geometry>
+        <box size="0.5 0.3 0.07"/>
+      </geometry>
+      <material name="blue"/>
+    </visual>
+    <!-- caster front -->
+    <!-- <collision name="caster_front_collision">
+      <origin rpy=" 0 0 0" xyz="0.35 0 -0.05"/>
+      <geometry>
+        <sphere radius="0.05"/>
+      </geometry>
+      <surface>
+        <friction>
+          <ode>
+            <mu>0</mu>
+            <mu2>0</mu2>
+            <slip1>1.0</slip1>
+            <slip2>1.0</slip2>
+          </ode>
+        </friction>
+      </surface>
+    </collision> -->
+    <visual name="caster_front_visual">
+      <origin rpy=" 0 0 0" xyz="0.2 0 -0.05"/>
+      <geometry>
+        <sphere radius="0.05"/>
+      </geometry>
+    </visual>
     </link>
-    <link name="link_left_wheel">
-        <inertial>
-            <mass value="0.2"/>
-            <origin rpy="0 1.5707 1.5707" xyz="0 0 0"/>
-            <inertia ixx="0.000526666666667" ixy="0" ixz="0" iyy="0.000526666666667" iyz="0" izz="0.001"/>
-        </inertial>
-        <collision name="link_left_wheel_collision">
-            <origin rpy="0 1.5707 1.5707" xyz="0 0 0"/>
-            <geometry>
-                <cylinder radius="0.04" length="0.01"/>
-            </geometry>
-        </collision>
-        <visual name="left_wheel" >
-            <origin xyz="0 0 0" rpy="0 1.5707 1.5707" />
-            <geometry>
-                <cylinder radius="0.04" length="0.01"/>
-            </geometry>
-        </visual>
-    </link>
-    <link name="link_right_wheel">
-        <inertial>
-            <mass value="0.2"/>
-            <origin rpy="0 1.5707 1.5707" xyz="0 0 0"/>
-            <inertia ixx="0.000526666666667" ixy="0" ixz="0" iyy="0.000526666666667" iyz="0" izz="0.001"/>
-        </inertial>
-        <collision name="link_right_wheel_collision">
-            <origin rpy="0 1.5707 1.5707" xyz="0 0 0"/>
-            <geometry>
-                <cylinder radius="0.04" length="0.01"/>
-            </geometry>
-        </collision>
-        <visual name="right_wheel" >
-            <origin xyz="0 0 0" rpy="0 1.5707 1.5707" />
-            <geometry>
-                <cylinder radius="0.04" length="0.01"/>
-            </geometry>
-        </visual>
-    </link>
-    <joint name="left_wheel_joint" type="continuous">
-        <parent link="link_base"/>
-        <child link="link_left_wheel"/>
-        <origin xyz="0 0.11 -0.02" rpy="0 0 0"/>
-        <axis xyz="0 1 0" rpy="0 0 0"/>
-        <limit effort="0.4" velocity="0.299"/>
-        <joint_properties damping="1.0" friction="1.0" />
-    </joint>
-    <joint name="right_wheel_joint" type="continuous">
-        <parent link="link_base"/>
-        <child link="link_right_wheel"/>
-        <origin xyz="0 -0.11 -0.02" rpy="0 0 0"/>
-        <axis xyz="0 1 0" rpy="0 0 0"/>
-        <limit effort="0.4" velocity="0.299"/>
-        <joint_properties damping="1.0" friction="1.0" />
-    </joint>
-    <transmission name="left_wheel_joint_trans" type="SimpleTransmission">
+  <!-- Create wheel right -->
+  <link name="right_wheel_link">
+    <inertial>
+      <mass value="0.2"/>
+      <origin rpy="0 1.5707 1.5707" xyz="0 0 0"/>
+      <inertia ixx="0.00052666666" ixy="0" ixz="0" iyy="0.00052666666" iyz="0" izz="0.001"/>
+    </inertial>
+    <collision name="link_right_wheel_collision">
+      <origin rpy="0 1.5707 1.5707" xyz="0 0 0" />
+      <geometry>
+        <cylinder length="0.04" radius="0.1"/>
+      </geometry>
+    </collision>
+    <visual name="link_right_wheel_visual">
+      <origin rpy="0 1.5707 1.5707" xyz="0 0 0"/>
+      <geometry>
+        <cylinder length="0.04" radius="0.1"/>
+      </geometry>
+    </visual>
+  </link>
+  <!--   Joint for right wheel  -->
+  <joint name="right_wheel_joint" type="continuous">
+    <origin rpy="0 0 0" xyz="-0.05 0.15 0"/>
+    <child link="right_wheel_link" />
+    <parent link="base_link"/>
+    <axis rpy="0 0 0" xyz="0 1 0"/>
+    <limit effort="10000" velocity="1000"/>
+    <joint_properties damping="1.0" friction="1.0" />
+  </joint>
+  <!-- Left Wheel link -->
+  <link name="left_wheel_link">
+    <inertial>
+      <mass value="0.2"/>
+      <origin rpy="0 1.5707 1.5707" xyz="0 0 0"/>
+      <inertia ixx="0.00052666666" ixy="0" ixz="0" iyy="0.00052666666" iyz="0" izz="0.001"/>
+    </inertial>
+    <collision name="link_left_wheel_collision">
+      <origin rpy="0 1.5707 1.5707" xyz="0 0 0" />
+      <geometry>
+        <cylinder length="0.04" radius="0.1"/>
+      </geometry>
+    </collision>
+    <visual name="link_left_wheel_visual">
+      <origin rpy="0 1.5707 1.5707" xyz="0 0 0"/>
+      <geometry>
+        <cylinder length="0.04" radius="0.1"/>
+      </geometry>
+    </visual>
+  </link>
+  <!--   Joint for right wheel  -->
+  <joint name="left_wheel_joint" type="continuous">
+    <origin rpy="0 0 0" xyz="-0.05 -0.15 0"/>
+    <child link="left_wheel_link" />
+    <parent link="base_link"/>
+    <axis rpy="0 0 0" xyz="0 1 0"/>
+    <limit effort="10000" velocity="1000"/>
+    <joint_properties damping="1.0" friction="1.0" />
+  </joint>
+  <transmission name="left_wheel_joint_trans" type="SimpleTransmission">
         <type>transmission_interface/SimpleTransmission</type>
         <joint name="left_wheel_joint">
