Commit message: update

File: src/vacumm_description/urdf/vacumm2.xacro (robot description, xacro)
@@ -5,9 +5,32 @@
         <turnGravityOff>false</turnGravityOff>
     </gazebo>
+    <gazebo reference="left_Wheel_link">
+        <mu1 value="1.0"/>
+        <mu2 value="1.0"/>
+        <kp value="600000"/>
+        <kd value="3"/>
+        <fdir1 value="1 0 0"/>
+        <material>Gazebo/Grey</material>
+        <turnGravityOff>false</turnGravityOff>
+    </gazebo>
+    <gazebo reference="right_Wheel_link">
+        <mu1 value="1.0"/>
+        <mu2 value="1.0"/>
+        <kp value="600000"/>
+        <kd value="3"/>
+        <fdir1 value="1 0 0"/>
+        <material>Gazebo/Grey</material>
+        <turnGravityOff>false</turnGravityOff>
+    </gazebo>
+    <gazebo>
+        <plugin name="gazebo_ros_control" filename="libgazebo_ros_control.so">
+            <legacyMode>false</legacyMode>
+        </plugin>
+    </gazebo>
     <link name="base_link">
         <pose>0 0 0.1 0 0 0</pose>
         <inertial>
             <mass value="2"/>
-            <origin rpy="0 0 0" xyz="0 0 0.1"/>
+            <origin rpy="0 0 0" xyz="0 0 0"/>
             <inertia ixx="0.0395416666667" ixy="0" ixz="0" iyy="0.106208333333" iyz="0" izz="0.106208333333"/>
         </inertial>
@@ -23,16 +46,16 @@
             </geometry>
         </visual>
-        <collision name="front_castor_holder_collision">
+        <!-- <collision name="front_castor_holder_collision">
             <origin rpy="0 0 0" xyz="0.15 0 -0.12"/>
             <geometry>
                 <cylinder radius="0.01" length="0.04"/>
             </geometry>
-        </collision>
-        <visual name="front_castor_holder">
+        </collision> -->
+        <!-- <visual name="front_castor_holder">
             <origin rpy="0 0 0" xyz="0.15 0 -0.12"/>
             <geometry>
                 <cylinder radius="0.01" length="0.04"/>
             </geometry>
-        </visual>
+        </visual> -->
         <collision name="front_castor_wheel_collision">
             <origin rpy="0 0 0" xyz="0.15 0 -0.14"/>
@@ -57,4 +80,5 @@
             </geometry>
         </visual>
+<!--
         <collision name="back_castor_holder_collision">
             <origin rpy="0 0 0" xyz="-0.15 0 -0.12"/>
@@ -62,11 +86,11 @@
                 <cylinder radius="0.01" length="0.04"/>
             </geometry>
-        </collision>
-        <visual name="back_castor_holder">
+        </collision> -->
+        <!-- <visual name="back_castor_holder">
             <origin rpy="0 0 0" xyz="-0.15 0 -0.12"/>
             <geometry>
                 <cylinder radius="0.01" length="0.04"/>
             </geometry>
-        </visual>
+        </visual> -->
         <collision name="back_castor_wheel_collision">
             <origin rpy="0 0 0" xyz="-0.15 0 -0.14"/>
@@ -92,3 +116,77 @@
         </visual>
     </link>
+    <link name="left_wheel_link">
+        <inertial>
+        <mass value="0.2"/>
+        <origin rpy="0 1.5707 1.5707" xyz="0 0 0"/>
+        <inertia ixx="0.000082" ixy="0" ixz="0" iyy="0.000082" iyz="0" izz="0.00016"/>
+        </inertial>
+        <collision name="link_left_wheel_collision">
+            <origin rpy="0 1.5707 1.5707" xyz="0 0 0" />
+            <geometry>
+                <cylinder length="0.01" radius="0.04"/>
+            </geometry>
+        </collision>
+        <visual name="link_left_wheel_visual">
+            <origin rpy="0 1.5707 1.5707" xyz="0 0 0"/>
+            <geometry>
+                <cylinder length="0.01" radius="0.04"/>
+            </geometry>
+        </visual>
+    </link>
+    <joint name="left_wheel_joint" type="continuous">
+        <origin rpy="0 0 0" xyz="0 -0.21 -0.125"/>
+        <child link="left_wheel_link" />
+        <parent link="base_link"/>
+        <axis rpy="0 0 0" xyz="0 1 0"/>
+        <limit effort="10000" velocity="1000"/>
+        <joint_properties damping="1.0" friction="1.0" />
+    </joint>
+    <link name="right_wheel_link">
+        <inertial>
+        <mass value="0.2"/>
+        <origin rpy="0 1.5707 1.5707" xyz="0 0 0"/>
+        <inertia ixx="0.000082" ixy="0" ixz="0" iyy="0.000082" iyz="0" izz="0.00016"/>
+        </inertial>
+        <collision name="link_right_wheel_collision">
+            <origin rpy="0 1.5707 1.5707" xyz="0 0 0" />
+            <geometry>
+                <cylinder length="0.01" radius="0.04"/>
+            </geometry>
+        </collision>
+        <visual name="link_right_wheel_visual">
+            <origin rpy="0 1.5707 1.5707" xyz="0 0 0"/>
+            <geometry>
+                <cylinder length="0.01" radius="0.04"/>
+            </geometry>
+        </visual>
+    </link>
+    <joint name="right_wheel_joint" type="continuous">
+        <origin rpy="0 0 0" xyz="0 0.21 -0.125"/>
+        <child link="right_wheel_link" />
+        <parent link="base_link"/>
+        <axis rpy="0 0 0" xyz="0 1 0"/>
+        <limit effort="10000" velocity="1000"/>
+        <joint_properties damping="1.0" friction="1.0" />
+    </joint>
+    <transmission name="left_wheel_joint_trans" type="SimpleTransmission">
+        <type>transmission_interface/SimpleTransmission</type>
+        <joint name="left_wheel_joint">
+            <hardwareInterface>hardware_interface/VelocityJointInterface</hardwareInterface>
+        </joint>
+        <actuator name="left_wheel_joint_motor">
+            <hardwareInterface>hardware_interface/VelocityJointInterface</hardwareInterface>
+            <mechanicalReduction>1</mechanicalReduction>
+        </actuator>
+    </transmission>
+    <transmission name="right_wheel_joint_trans" type="SimpleTransmission">
+        <type>transmission_interface/SimpleTransmission</type>
+        <joint name="right_wheel_joint">
+            <hardwareInterface>hardware_interface/VelocityJointInterface</hardwareInterface>
+        </joint>
+        <actuator name="right_wheel_joint_motor">
+            <hardwareInterface>hardware_interface/VelocityJointInterface</hardwareInterface>
+            <mechanicalReduction>1</mechanicalReduction>
+        </actuator>
+    </transmission>
 </robot>

Commit message: update

File: src/vacumm_description/urdf/vacumm2.xacro (robot description, xacro)
@@ -33,5 +33,5 @@
             <mass value="2"/>
             <origin rpy="0 0 0" xyz="0 0 0"/>
-            <inertia ixx="0.0395416666667" ixy="0" ixz="0" iyy="0.106208333333" iyz="0" izz="0.106208333333"/>
+            <inertia ixx="0.026667" ixy="0" ixz="0" iyy="0.026667" iyz="0" izz="0.04"/>
         </inertial>
         <collision name="chassis_collision">
