Commit message: update

File: src/vacumm_description/urdf/vacumm4.xacro (robot description, xacro)
@@ -64,20 +64,18 @@
   <xacro:macro name="gazebo_wheel" params="prefix">
     <gazebo reference="${prefix}_wheel">
-      <kp>1000000.0</kp>
-    <kd>100.0</kd>
-    <mu1>1.5</mu1>
-    <mu2>1.5</mu2>
-    <fdir1>1 0 0</fdir1>
-    <maxVel>1.0</maxVel>
-    <minDepth>0.00</minDepth>
-      <material>Gazebo/Grey</material>
-      <turnGravityOff>false</turnGravityOff>
+        <!-- <kp>1000000.0</kp>
+        <kd>1.0</kd> -->
+        <mu1>1.5</mu1>
+        <mu2>1.5</mu2>
+        <slip1>0</slip1>
+        <slip2>0</slip2>
+        <!-- <minDepth>0.01</minDepth> -->
+        <material>Gazebo/Grey</material>
+        <turnGravityOff>false</turnGravityOff>
     </gazebo>
   </xacro:macro>
   <gazebo reference="base_link">
-    <mu1 value="0"/>
-    <mu2 value="0"/>
-     <kp>1000000.0</kp>
-    <kd>100.0</kd>
+    <!-- <mu1 value="0"/>
+    <mu2 value="0"/> -->
     <material>Gazebo/Grey</material>
     <turnGravityOff>false</turnGravityOff>
@@ -87,8 +85,6 @@
       <mu1 value="0"/>
       <mu2 value="0"/>
-      <erp value="0"/>
-      <fdir1 value="1 1 1"/>
-      <slip1 value="1"/>
-      <slip2 value="1"/>
+      <!-- <slip1 value="1"/>
+      <slip2 value="1"/> -->
       <material>Gazebo/Grey</material>
       <turnGravityOff>false</turnGravityOff>
@@ -152,4 +148,25 @@
     <plugin name="gazebo_ros_control" filename="libgazebo_ros_control.so">
       <legacyMode>false</legacyMode>
+    </plugin>
+  </gazebo>
+<gazebo>
+    <plugin filename="libgazebo_ros_diff_drive.so" name="differential_drive_controller">
+      <alwaysOn>true</alwaysOn>
+      <updateRate>20</updateRate>
+      <leftJoint>left_wheel_joint</leftJoint>
+      <rightJoint>right_wheel_joint</rightJoint>
+      <wheelSeparation>0.235</wheelSeparation>
+      <wheelDiameter>0.08</wheelDiameter>
+      <torque>0.1</torque>
+      <commandTopic>cmd_vel</commandTopic>
+      <odometryTopic>odom</odometryTopic>
+      <odometryFrame>odom</odometryFrame>
+      <odometrySource>1</odometrySource>
+        <publishOdomTF>true</publishOdomTF>
+    <robotBaseFrame>base_footprint</robotBaseFrame>
+    <publishWheelTF>false</publishWheelTF>
+    <publishTf>true</publishTf>
+    <publishWheelJointState>false</publishWheelJointState>
+    <legacyMode>false</legacyMode>
     </plugin>
   </gazebo>

Commit message: update

File: src/vacumm_description/urdf/vacumm4.xacro (robot description, xacro)
@@ -286,10 +286,10 @@
   <xacro:wheel_transmission prefix="right" />
   <xacro:macro name="sensor_kinect" params="parent">
-    <joint name="camera_rgb_joint" type="fixed">
+    <joint name="camera_joint" type="fixed">
       <origin xyz="${cam_px} ${kinect_cam_py} ${cam_pz}" rpy="${cam_or} ${cam_op} ${cam_oy}"/>
       <parent link="${parent}"/>
-      <child link="camera_rgb_frame" />
-    </joint>
-    <link name="camera_rgb_frame"/>
+      <child link="camera_link" />
+    </joint>
+    <link name="camera_link"/>
     <joint name="camera_rgb_optical_joint" type="fixed">
       <origin xyz="0 0 0" rpy="${-M_PI/2} 0 ${-M_PI/2}" />
@@ -298,10 +298,10 @@
     </joint>
     <link name="camera_rgb_optical_frame"/>
-    <joint name="camera_joint" type="fixed">
+    <joint name="camera_rgb_joint" type="fixed">
       <origin xyz="-0.031 ${-kinect_cam_py} -0.016" rpy="0 0 0"/>
-      <parent link="camera_rgb_frame"/>
-      <child link="camera_link"/>
-    </joint>
-    <link name="camera_link">
+      <parent link="camera_link"/>
+      <child link="camera_rgb_frame"/>
+    </joint>
+    <link name="camera_rgb_frame">
       <visual>
         <origin xyz="0 0 0" rpy="0 0 ${M_PI/2}"/>
