Commit message: update

File: src/vacumm_description/urdf/vacumm5.xacro (robot description, xacro)
@@ -2,13 +2,11 @@
 <robot xmlns:xacro="http://www.ros.org/wiki/xacro" name="kbot">
   <xacro:property name="base_width" value="0.2"/>
-  <xacro:property name="base_len" value="0.16"/>
+  <xacro:property name="base_len" value="0.15"/>
   <xacro:property name="wheel_radius" value="0.04"/>
   <xacro:property name="base_wheel_gap" value="0.0175"/>
-  <xacro:property name="wheel_joint_offset" value="0"/>
-  <xacro:property name="wheel_joint_drop_offset" value="-0.02"/>
+  <xacro:property name="wheel_joint_offset" value="0.02"/>
   <xacro:property name="caster_wheel_radius" value="${wheel_radius/2}"/>
   <xacro:property name="caster_wheel_mass" value="0.001"/>
-  <xacro:property name="caster_wheel_joint_offset" value="0.07"/>
-  <xacro:property name="caster_wheel_down_offset" value="0.0001"/>
+  <xacro:property name="caster_wheel_joint_offset" value="-0.052"/>
     <xacro:property name="M_PI" value="3.1415926535897931" />
     <xacro:property name="cam_px" value="0.025" />
@@ -31,95 +29,8 @@
     <color rgba="0.8 0.0 0.0 1.0"/>
   </material>
-  <!--Interial macros-->
-  <xacro:macro name="cylinder_inertia" params="m r h">
-    <inertial>
-      <mass value="${m}"/>
-      <inertia ixx="${m*(3*r*r+h*h)/12}" ixy = "0" ixz = "0" iyy="${m*(3*r*r+h*h)/12}" iyz = "0" izz="${m*r*r/2}"/>
-    </inertial>
-  </xacro:macro>
-  <xacro:macro name="box_inertia" params="m w h d">
-    <inertial>
-      <mass value="${m}"/>
-      <inertia ixx="${m / 12.0 * (d*d + h*h)}" ixy="0.0" ixz="0.0" iyy="${m / 12.0 * (w*w + h*h)}" iyz="0.0" izz="${m / 12.0 * (w*w + d*d)}"/>
-    </inertial>
-  </xacro:macro>
-  <xacro:macro name="sphere_inertia" params="m r">
-    <inertial>
-      <mass value="${m}"/>
-      <inertia ixx="${2.0*m*(r*r)/5.0}" ixy="0.0" ixz="0.0" iyy="${2.0*m*(r*r)/5.0}" iyz="0.0" izz="${2.0*m*(r*r)/5.0}"/>
-    </inertial>
-  </xacro:macro>
-  <xacro:macro name="wheel_transmission" params="prefix">
-        <transmission name="${prefix}_wheel_joint_trans" type="SimpleTransmission">
-            <type>transmission_interface/SimpleTransmission</type>
-            <joint name="${prefix}_wheel_joint">
-                <hardwareInterface>hardware_interface/VelocityJointInterface</hardwareInterface>
-            </joint>
-            <actuator name="${prefix}_wheel_joint_motor">
-                <hardwareInterface>hardware_interface/VelocityJointInterface</hardwareInterface>
-                <mechanicalReduction>1</mechanicalReduction>
-            </actuator>
-        </transmission>
-    </xacro:macro>
-  <xacro:macro name="gazebo_wheel" params="prefix">
-    <gazebo reference="${prefix}_wheel">
-        <!-- <mu1 value="1.16"/>
-        <mu2 value="1.16"/> -->
-        <material>Gazebo/Grey</material>
-        <!-- <turnGravityOff>false</turnGravityOff> -->
-    </gazebo>
-  </xacro:macro>
-    <gazebo reference="base_link">
-        <material>Gazebo/Grey</material>
-        <turnGravityOff>false</turnGravityOff>
-    </gazebo>
-  <!-- <xacro:macro name="gazebo_caster" params="prefix">
-    <gazebo reference="${prefix}_caster_wheel">
-        <mu1 value="1.16"/>
-        <mu2 value="1.16"/>
-        <material>Gazebo/Grey</material>
-        <turnGravityOff>false</turnGravityOff>
-    </gazebo>
-  </xacro:macro> -->
-    <xacro:macro name="wheel_transmission" params="prefix">
-        <transmission name="${prefix}_wheel_joint_trans" type="SimpleTransmission">
-            <type>transmission_interface/SimpleTransmission</type>
-            <joint name="${prefix}_wheel_joint">
-                <hardwareInterface>hardware_interface/VelocityJointInterface</hardwareInterface>
-            </joint>
-            <actuator name="${prefix}_wheel_joint_motor">
-                <hardwareInterface>hardware_interface/VelocityJointInterface</hardwareInterface>
-                <mechanicalReduction>1</mechanicalReduction>
-            </actuator>
-        </transmission>
-    </xacro:macro>
-<!--Front Caster Wheel Link-->
-  <xacro:macro name="caster_wheel" params="prefix reflect">
-      <collision>
-        <origin xyz="${caster_wheel_joint_offset*reflect} 0 -${((base_width/2))-caster_wheel_down_offset}" rpy="0 0 0"/>
-        <geometry>
-          <sphere radius="${caster_wheel_radius}"/>
-        </geometry>
-        <surface>
-          <friction>
-            <ode>
-              <mu>0</mu>
-              <mu2>0</mu2>
-              <slip1>0</slip1>
-              <slip2>0</slip2>
-            </ode>
-          </friction>
-        </surface>
-      </collision>
-      <xacro:sphere_inertia m="0.02" r="${caster_wheel_radius}"/>
-  </xacro:macro>
-    <!-- <xacro:gazebo_wheel prefix="left"/>
-    <xacro:gazebo_wheel prefix="right"/>
-    <xacro:gazebo_caster prefix="front"/>
-    <xacro:gazebo_caster prefix="back"/> -->
-    <gazebo>
-        <plugin name="gazebo_ros_control" filename="libgazebo_ros_control.so">
-            <legacyMode>false</legacyMode>
-        </plugin>
+  <gazebo>
+      <plugin name="gazebo_ros_control" filename="libgazebo_ros_control.so">
+          <legacyMode>false</legacyMode>
+      </plugin>
     </gazebo>
     <xacro:macro name="vacumm_sim_3dsensor">
@@ -161,7 +72,26 @@
     </gazebo>
   </xacro:macro>
+  <!--Interial macros-->
+  <xacro:macro name="cylinder_inertia" params="m r h">
+    <inertial>
+      <mass value="${m}"/>
+      <inertia ixx="${m*(3*r*r+h*h)/12}" ixy = "0" ixz = "0" iyy="${m*(3*r*r+h*h)/12}" iyz = "0" izz="${m*r*r/2}"/>
+    </inertial>
+  </xacro:macro>
+  <xacro:macro name="box_inertia" params="m w h d">
+    <inertial>
+      <mass value="${m}"/>
+      <inertia ixx="${m / 12.0 * (d*d + h*h)}" ixy="0.0" ixz="0.0" iyy="${m / 12.0 * (w*w + h*h)}" iyz="0.0" izz="${m / 12.0 * (w*w + d*d)}"/>
+    </inertial>
+  </xacro:macro>
+  <xacro:macro name="sphere_inertia" params="m r">
+    <inertial>
+      <mass value="${m}"/>
+      <inertia ixx="${2.0*m*(r*r)/5.0}" ixy="0.0" ixz="0.0" iyy="${2.0*m*(r*r)/5.0}" iyz="0.0" izz="${2.0*m*(r*r)/5.0}"/>
+    </inertial>
+  </xacro:macro>
   <!--Base Footprint-->
   <link name="base_footprint">
-    <xacro:box_inertia m="1" w="0.001" h="0.001" d="0.001"/>
+    <xacro:box_inertia m="10" w="0.001" h="0.001" d="0.001"/>
     <visual>
         <origin xyz="0 0 0" rpy="0 0 0" />
@@ -173,8 +103,8 @@
   <!--Base link-->
   <link name="base_link">
-    <xacro:cylinder_inertia m="1" r="${base_width/2}" h="${base_len}"/>
+    <xacro:box_inertia m="1" w="${base_len}" h="${base_width}" d="0.01"/>
     <visual>
       <geometry>
-        <cylinder radius="${base_width/2}" length="${base_len}"/>
+        <box size="${base_len} ${base_width} 0.01"/>
       </geometry>
       <material name="black"/>
@@ -182,13 +112,11 @@
     <collision>
       <geometry>
-        <cylinder radius="${base_width/2}" length="${base_len}"/>
+        <box size="${base_len} ${base_width} 0.01"/>
       </geometry>
     </collision>
-    <xacro:caster_wheel prefix="front" reflect="1"/>
-    <xacro:caster_wheel prefix="back" reflect="-1"/>
   </link>
   <!--base_link to base_footprint Joint-->
   <joint name="base_link_joint" type="fixed">
-    <origin xyz="0 0 0" rpy="0 0 0" />
+    <origin xyz="0 0 ${wheel_radius + 0.005}" rpy="0 0 0" />
     <parent link="base_footprint"/>
     <child link="base_link" />
@@ -210,5 +138,5 @@
         </geometry>
       </collision>
-      <xacro:cylinder_inertia m="3" r="${wheel_radius}" h="0.005"/>
+      <xacro:cylinder_inertia m="1" r="${wheel_radius}" h="0.005"/>
     </link>
     <joint name="${prefix}_wheel_joint" type="continuous">
@@ -216,7 +144,5 @@
       <parent link="base_link"/>
       <child link="${prefix}_wheel"/>
-      <limit effort="10000" velocity="1000"/>
-      <joint_properties damping="1.0" friction="1.0" />
-      <origin xyz="${wheel_joint_offset} ${((base_width/2)+base_wheel_gap)*reflect} -${(base_width/2)+wheel_joint_drop_offset}" rpy="0 0 0"/>
+      <origin xyz="${wheel_joint_offset} ${((base_width/2)+base_wheel_gap)*reflect} -0.005" rpy="0 0 0"/>
     </joint>
   </xacro:macro>
@@ -224,7 +150,43 @@
   <xacro:wheel prefix="left" reflect="1"/>
   <xacro:wheel prefix="right" reflect="-1"/>
-  <xacro:wheel_transmission prefix="left" />
-  <xacro:wheel_transmission prefix="right" />
-  <xacro:macro name="sensor_kinect" params="parent">
+  <!--Caster Wheel Link-->
+  <link name="caster_wheel">
+    <visual>
+      <origin xyz="0 0 0" rpy="0 0 0"/>
+      <geometry>
+        <sphere radius="${caster_wheel_radius}"/>
+      </geometry>
+      <material name="blue"/>
+    </visual>
+    <collision>
+      <origin xyz="0 0 0" rpy="0 0 0"/>
+      <geometry>
+        <sphere radius="${caster_wheel_radius}"/>
+      </geometry>
+    </collision>
+    <xacro:sphere_inertia m="1" r="${caster_wheel_radius}"/>
+  </link>
+  <!--Caster Wheel Joint-->
+  <joint name="caster_wheel_joint" type="continuous">
+    <axis xyz="0 1 0" rpy="0 0 0" />
+    <parent link="base_link"/>
+    <child link="caster_wheel"/>
+    <origin xyz="${caster_wheel_joint_offset} 0 -${caster_wheel_radius+0.005}" rpy="0 0 0"/>
+  </joint>
+  <xacro:macro name="wheel_transmission" params="prefix">
+        <transmission name="${prefix}_wheel_joint_trans" type="SimpleTransmission">
+            <type>transmission_interface/SimpleTransmission</type>
+            <joint name="${prefix}_wheel_joint">
+                <hardwareInterface>hardware_interface/VelocityJointInterface</hardwareInterface>
+            </joint>
+            <actuator name="${prefix}_wheel_joint_motor">
+                <hardwareInterface>hardware_interface/VelocityJointInterface</hardwareInterface>
+                <mechanicalReduction>1</mechanicalReduction>
+            </actuator>
+        </transmission>
+    </xacro:macro>
+    <xacro:wheel_transmission prefix="left" />
+    <xacro:wheel_transmission prefix="right" />
+    <xacro:macro name="sensor_kinect" params="parent">
     <joint name="camera_rgb_joint" type="fixed">
       <origin xyz="${cam_px} ${kinect_cam_py} ${cam_pz}" rpy="${cam_or} ${cam_op} ${cam_oy}"/>
