Commit message: update

File: src/vacumm_description/urdf/vacumm5.xacro (robot description, xacro)
@@ -1,19 +1,21 @@
 <?xml version="1.0"?>
-<robot xmlns:xacro="http://www.ros.org/wiki/xacro" name="kbot">
+<robot xmlns:xacro="http://www.ros.org/wiki/xacro" name="vacumm_bot1">
   <xacro:property name="base_width" value="0.2"/>
-  <xacro:property name="base_len" value="0.15"/>
+  <xacro:property name="base_len" value="0.16"/>
   <xacro:property name="wheel_radius" value="0.04"/>
   <xacro:property name="base_wheel_gap" value="0.0175"/>
-  <xacro:property name="wheel_joint_offset" value="0.02"/>
+  <xacro:property name="wheel_joint_offset" value="0"/>
+  <xacro:property name="wheel_joint_drop_offset" value="-0.02"/>
   <xacro:property name="caster_wheel_radius" value="${wheel_radius/2}"/>
-  <xacro:property name="caster_wheel_mass" value="0.001"/>
-  <xacro:property name="caster_wheel_joint_offset" value="-0.052"/>
-    <xacro:property name="M_PI" value="3.1415926535897931" />
-    <xacro:property name="cam_px" value="0.025" />
-    <xacro:property name="cam_pz" value="${base_len-0.025}" />
-    <xacro:property name="kinect_cam_py" value="0"/>
-    <xacro:property name="cam_or" value="0" />
-	<xacro:property name="cam_op" value="0" />
-	<xacro:property name="cam_oy" value="0" />
+  <xacro:property name="caster_wheel_mass" value="0.0001"/>
+  <xacro:property name="caster_wheel_joint_offset" value="0.07"/>
+  <xacro:property name="caster_wheel_down_offset" value="0.0001"/>
+  <xacro:property name="M_PI" value="3.1415926535897931" />
+  <xacro:property name="cam_px" value="0.025" />
+  <xacro:property name="cam_pz" value="${base_len-0.025}" />
+  <xacro:property name="kinect_cam_py" value="0"/>
+  <xacro:property name="cam_or" value="0" />
+  <xacro:property name="cam_op" value="0" />
+  <xacro:property name="cam_oy" value="0" />
   <!--Color Properties-->
   <material name="blue">
@@ -29,10 +31,145 @@
     <color rgba="0.8 0.0 0.0 1.0"/>
   </material>
-  <gazebo>
-      <plugin name="gazebo_ros_control" filename="libgazebo_ros_control.so">
-          <legacyMode>false</legacyMode>
-      </plugin>
+  <!--Interial macros-->
+  <xacro:macro name="cylinder_inertia" params="m r h">
+    <inertial>
+      <mass value="${m}"/>
+      <inertia ixx="${m*(3*r*r+h*h)/12}" ixy = "0" ixz = "0" iyy="${m*(3*r*r+h*h)/12}" iyz = "0" izz="${m*r*r/2}"/>
+    </inertial>
+  </xacro:macro>
+  <xacro:macro name="box_inertia" params="m w h d">
+    <inertial>
+      <mass value="${m}"/>
+      <inertia ixx="${m / 12.0 * (d*d + h*h)}" ixy="0.0" ixz="0.0" iyy="${m / 12.0 * (w*w + h*h)}" iyz="0.0" izz="${m / 12.0 * (w*w + d*d)}"/>
+    </inertial>
+  </xacro:macro>
+  <xacro:macro name="sphere_inertia" params="m r">
+    <inertial>
+      <mass value="${m}"/>
+      <inertia ixx="${2.0*m*(r*r)/5.0}" ixy="0.0" ixz="0.0" iyy="${2.0*m*(r*r)/5.0}" iyz="0.0" izz="${2.0*m*(r*r)/5.0}"/>
+    </inertial>
+  </xacro:macro>
+  <xacro:macro name="wheel_transmission" params="prefix">
+    <transmission name="${prefix}_wheel_joint_trans" type="SimpleTransmission">
+      <type>transmission_interface/SimpleTransmission</type>
+      <joint name="${prefix}_wheel_joint">
+        <hardwareInterface>hardware_interface/VelocityJointInterface</hardwareInterface>
+      </joint>
+      <actuator name="${prefix}_wheel_joint_motor">
+        <hardwareInterface>hardware_interface/VelocityJointInterface</hardwareInterface>
+        <mechanicalReduction>1</mechanicalReduction>
+      </actuator>
+    </transmission>
+  </xacro:macro>
+  <xacro:macro name="gazebo_wheel" params="prefix">
+    <gazebo reference="${prefix}_wheel">
+        <!-- <kp>1000000.0</kp>
+        <kd>1.0</kd> -->
+        <mu1>1.5</mu1>
+        <mu2>1.5</mu2>
+        <slip1>0</slip1>
+        <slip2>0</slip2>
+        <!-- <minDepth>0.01</minDepth> -->
+        <material>Gazebo/Grey</material>
+        <turnGravityOff>false</turnGravityOff>
     </gazebo>
-    <xacro:macro name="vacumm_sim_3dsensor">
+  </xacro:macro>
+  <gazebo reference="base_link">
+    <!-- <mu1 value="0"/>
+    <mu2 value="0"/> -->
+    <material>Gazebo/Grey</material>
+    <turnGravityOff>false</turnGravityOff>
+  </gazebo>
+  <xacro:macro name="gazebo_caster" params="prefix">
+    <gazebo reference="${prefix}_caster_wheel_link">
+      <mu1 value="0"/>
+      <mu2 value="0"/>
+      <!-- <slip1 value="1"/>
+      <slip2 value="1"/> -->
+      <material>Gazebo/Grey</material>
+      <turnGravityOff>false</turnGravityOff>
+    </gazebo>
+  </xacro:macro>
+  <xacro:gazebo_wheel prefix="left"/>
+  <xacro:gazebo_wheel prefix="right"/>
+  <xacro:gazebo_caster prefix="front"/>
+  <xacro:gazebo_caster prefix="back"/>
+  <xacro:macro name="wheel_transmission" params="prefix">
+    <transmission name="${prefix}_wheel_joint_trans" type="SimpleTransmission">
+      <type>transmission_interface/SimpleTransmission</type>
+      <joint name="${prefix}_wheel_joint">
+        <hardwareInterface>hardware_interface/VelocityJointInterface</hardwareInterface>
+      </joint>
+      <actuator name="${prefix}_wheel_joint_motor">
+        <hardwareInterface>hardware_interface/VelocityJointInterface</hardwareInterface>
+        <mechanicalReduction>1</mechanicalReduction>
+      </actuator>
+    </transmission>
+  </xacro:macro>
+  <!--Front Caster Wheel Link-->
+  <xacro:macro name="caster_wheel" params="prefix reflect">
+    <!--Caster Wheel Link-->
+    <link name="${prefix}_caster_wheel_link">
+      <!-- <visual>
+      <origin xyz="0 0 0" rpy="0 0 0"/>
+      <geometry>
+        <sphere radius="${caster_wheel_radius}"/>
+      </geometry>
+      <material name="blue"/>
+    </visual> -->
+      <collision >
+        <origin xyz="0 0 0" rpy="0 0 0"/>
+        <geometry>
+          <sphere radius="${caster_wheel_radius}"/>
+        </geometry>
+        <surface>
+          <friction>
+            <ode>
+              <mu>0</mu>
+              <mu2>0</mu2>
+              <slip1>1</slip1>
+              <slip2>1</slip2>
+            </ode>
+          </friction>
+        </surface>
+      </collision>
+      <xacro:sphere_inertia m="0.02" r="${caster_wheel_radius}"/>
+    </link>
+    <!--Caster Wheel Joint-->
+    <joint name="${prefix}_caster_wheel_joint" type="continuous">
+      <axis xyz="0 1 0" rpy="0 0 0" />
+      <parent link="base_link"/>
+      <child link="${prefix}_caster_wheel_link"/>
+      <origin xyz="${caster_wheel_joint_offset*reflect} 0 -${((base_width/2))-caster_wheel_down_offset}" rpy="0 0 0"/>
+    </joint>
+    <xacro:sphere_inertia m="0.02" r="${caster_wheel_radius}"/>
+  </xacro:macro>
+  <!-- <gazebo>
+    <plugin name="gazebo_ros_control" filename="libgazebo_ros_control.so">
+      <legacyMode>false</legacyMode>
+    </plugin>
+  </gazebo> -->
+<!-- <gazebo>
+    <plugin filename="libgazebo_ros_diff_drive.so" name="differential_drive_controller">
+      <alwaysOn>true</alwaysOn>
+      <updateRate>20</updateRate>
+      <leftJoint>left_wheel_joint</leftJoint>
+      <rightJoint>right_wheel_joint</rightJoint>
+      <wheelSeparation>0.235</wheelSeparation>
+      <wheelDiameter>0.08</wheelDiameter>
+      <torque>0.1</torque>
+      <commandTopic>cmd_vel</commandTopic>
+      <odometryTopic>odom</odometryTopic>
+      <odometryFrame>odom</odometryFrame>
+      <odometrySource>1</odometrySource>
+        <publishOdomTF>true</publishOdomTF>
+    <robotBaseFrame>base_footprint</robotBaseFrame>
+    <publishWheelTF>false</publishWheelTF>
+    <publishTf>true</publishTf>
+    <publishWheelJointState>false</publishWheelJointState>
+    <legacyMode>false</legacyMode>
+    </plugin>
+  </gazebo> -->
+  <xacro:macro name="vacumm_sim_3dsensor">
     <gazebo reference="camera_link">
       <sensor type="depth" name="camera">
@@ -72,39 +209,20 @@
     </gazebo>
   </xacro:macro>
-  <!--Interial macros-->
-  <xacro:macro name="cylinder_inertia" params="m r h">
-    <inertial>
-      <mass value="${m}"/>
-      <inertia ixx="${m*(3*r*r+h*h)/12}" ixy = "0" ixz = "0" iyy="${m*(3*r*r+h*h)/12}" iyz = "0" izz="${m*r*r/2}"/>
-    </inertial>
-  </xacro:macro>
-  <xacro:macro name="box_inertia" params="m w h d">
-    <inertial>
-      <mass value="${m}"/>
-      <inertia ixx="${m / 12.0 * (d*d + h*h)}" ixy="0.0" ixz="0.0" iyy="${m / 12.0 * (w*w + h*h)}" iyz="0.0" izz="${m / 12.0 * (w*w + d*d)}"/>
-    </inertial>
-  </xacro:macro>
-  <xacro:macro name="sphere_inertia" params="m r">
-    <inertial>
-      <mass value="${m}"/>
-      <inertia ixx="${2.0*m*(r*r)/5.0}" ixy="0.0" ixz="0.0" iyy="${2.0*m*(r*r)/5.0}" iyz="0.0" izz="${2.0*m*(r*r)/5.0}"/>
-    </inertial>
-  </xacro:macro>
   <!--Base Footprint-->
   <link name="base_footprint">
-    <xacro:box_inertia m="10" w="0.001" h="0.001" d="0.001"/>
+    <xacro:box_inertia m="1" w="0.001" h="0.001" d="0.001"/>
     <visual>
-        <origin xyz="0 0 0" rpy="0 0 0" />
-        <geometry>
-            <box size="0.001 0.001 0.001" />
-        </geometry>
+      <origin xyz="0 0 0" rpy="0 0 0" />
+      <geometry>
+        <box size="0.001 0.001 0.001" />
+      </geometry>
     </visual>
   </link>
   <!--Base link-->
   <link name="base_link">
-    <xacro:box_inertia m="1" w="${base_len}" h="${base_width}" d="0.01"/>
+    <xacro:cylinder_inertia m="1" r="${base_width/2}" h="${base_len}"/>
     <visual>
       <geometry>
-        <box size="${base_len} ${base_width} 0.01"/>
+        <cylinder radius="${base_width/2}" length="${base_len}"/>
       </geometry>
       <material name="black"/>
@@ -112,5 +230,5 @@
     <collision>
       <geometry>
-        <box size="${base_len} ${base_width} 0.01"/>
+        <cylinder radius="${base_width/2}" length="${base_len}"/>
       </geometry>
     </collision>
@@ -118,8 +236,10 @@
   <!--base_link to base_footprint Joint-->
   <joint name="base_link_joint" type="fixed">
-    <origin xyz="0 0 ${wheel_radius + 0.005}" rpy="0 0 0" />
+    <origin xyz="0 0 0" rpy="0 0 0" />
     <parent link="base_footprint"/>
     <child link="base_link" />
   </joint>
+  <xacro:caster_wheel prefix="front" reflect="1"/>
+  <xacro:caster_wheel prefix="back" reflect="-1"/>
   <!--Wheel link & joint macro-->
   <xacro:macro name="wheel" params="prefix reflect">
@@ -128,5 +248,5 @@
         <origin xyz="0 0 0" rpy="${pi/2} 0 0"/>
         <geometry>
-          <cylinder radius="${wheel_radius}" length="0.005"/>
+          <cylinder radius="${wheel_radius}" length="0.01"/>
         </geometry>
         <material name="red"/>
@@ -135,8 +255,19 @@
         <origin xyz="0 0 0" rpy="${pi/2} 0 0"/>
         <geometry>
-          <cylinder radius="${wheel_radius}" length="0.005"/>
-        </geometry>
+          <cylinder radius="${wheel_radius}" length="0.01"/>
+        </geometry>
+        <surface>
+          <friction>
+            <ode>
+              <mu>1.16</mu>
+              <mu2>1.16</mu2>
+              <fdir1>1 1 0</fdir1>
+              <slip1>0</slip1>
+              <slip2>0</slip2>
+            </ode>
+          </friction>
+        </surface>
       </collision>
-      <xacro:cylinder_inertia m="1" r="${wheel_radius}" h="0.005"/>
+      <xacro:sphere_inertia m="3" r="${wheel_radius}" />
     </link>
     <joint name="${prefix}_wheel_joint" type="continuous">
@@ -144,5 +275,7 @@
       <parent link="base_link"/>
       <child link="${prefix}_wheel"/>
-      <origin xyz="${wheel_joint_offset} ${((base_width/2)+base_wheel_gap)*reflect} -0.005" rpy="0 0 0"/>
+      <limit effort="10000" velocity="1000"/>
+      <joint_properties damping="0" friction="1.16" />
+      <origin xyz="${wheel_joint_offset} ${((base_width/2)+base_wheel_gap)*reflect} -${(base_width/2)+wheel_joint_drop_offset}" rpy="0 0 0"/>
     </joint>
   </xacro:macro>
@@ -150,49 +283,13 @@
   <xacro:wheel prefix="left" reflect="1"/>
   <xacro:wheel prefix="right" reflect="-1"/>
-  <!--Caster Wheel Link-->
-  <link name="caster_wheel">
-    <visual>
-      <origin xyz="0 0 0" rpy="0 0 0"/>
-      <geometry>
-        <sphere radius="${caster_wheel_radius}"/>
-      </geometry>
-      <material name="blue"/>
-    </visual>
-    <collision>
-      <origin xyz="0 0 0" rpy="0 0 0"/>
-      <geometry>
-        <sphere radius="${caster_wheel_radius}"/>
-      </geometry>
-    </collision>
-    <xacro:sphere_inertia m="1" r="${caster_wheel_radius}"/>
-  </link>
-  <!--Caster Wheel Joint-->
-  <joint name="caster_wheel_joint" type="continuous">
-    <axis xyz="0 1 0" rpy="0 0 0" />
-    <parent link="base_link"/>
-    <child link="caster_wheel"/>
-    <origin xyz="${caster_wheel_joint_offset} 0 -${caster_wheel_radius+0.005}" rpy="0 0 0"/>
-  </joint>
-  <xacro:macro name="wheel_transmission" params="prefix">
-        <transmission name="${prefix}_wheel_joint_trans" type="SimpleTransmission">
-            <type>transmission_interface/SimpleTransmission</type>
-            <joint name="${prefix}_wheel_joint">
-                <hardwareInterface>hardware_interface/VelocityJointInterface</hardwareInterface>
-            </joint>
-            <actuator name="${prefix}_wheel_joint_motor">
-                <hardwareInterface>hardware_interface/VelocityJointInterface</hardwareInterface>
-                <mechanicalReduction>1</mechanicalReduction>
-            </actuator>
-        </transmission>
-    </xacro:macro>
-    <xacro:wheel_transmission prefix="left" />
-    <xacro:wheel_transmission prefix="right" />
-    <xacro:macro name="sensor_kinect" params="parent">
-    <joint name="camera_rgb_joint" type="fixed">
+  <xacro:wheel_transmission prefix="left" />
+  <xacro:wheel_transmission prefix="right" />
+  <xacro:macro name="sensor_kinect" params="parent">
+    <joint name="camera_joint" type="fixed">
       <origin xyz="${cam_px} ${kinect_cam_py} ${cam_pz}" rpy="${cam_or} ${cam_op} ${cam_oy}"/>
       <parent link="${parent}"/>
-      <child link="camera_rgb_frame" />
-    </joint>
-    <link name="camera_rgb_frame"/>
+      <child link="camera_link" />
+    </joint>
+    <link name="camera_link"/>
     <joint name="camera_rgb_optical_joint" type="fixed">
       <origin xyz="0 0 0" rpy="${-M_PI/2} 0 ${-M_PI/2}" />
@@ -201,28 +298,26 @@
     </joint>
     <link name="camera_rgb_optical_frame"/>
-    <joint name="camera_joint" type="fixed">
+    <joint name="camera_rgb_joint" type="fixed">
       <origin xyz="-0.031 ${-kinect_cam_py} -0.016" rpy="0 0 0"/>
-      <parent link="camera_rgb_frame"/>
-      <child link="camera_link"/>
-    </joint>
-      <link name="camera_link">
+      <parent link="camera_link"/>
+      <child link="camera_rgb_frame"/>
+    </joint>
+    <link name="camera_rgb_frame">
       <visual>
-       <origin xyz="0 0 0" rpy="0 0 ${M_PI/2}"/>
-        <geometry>
-         <mesh filename="package://vacumm_description/meshes/sensors/kinect.dae"/>
+        <origin xyz="0 0 0" rpy="0 0 ${M_PI/2}"/>
+        <geometry>
+          <mesh filename="package://vacumm_description/meshes/sensors/kinect.dae"/>
         </geometry>
       </visual>
-  	  <collision>
+      <collision>
         <origin xyz="0.0 0.0 0.0" rpy="0 0 0"/>
-  	    <geometry>
-  	      <box size="0.07271 0.27794 0.073"/>
-  	    </geometry>
-  	  </collision>
+        <geometry>
+          <box size="0.07271 0.27794 0.073"/>
+        </geometry>
+      </collision>
       <inertial>
         <mass value="0.564" />
         <origin xyz="0 0 0" />
-        <inertia ixx="0.003881243" ixy="0.0" ixz="0.0"
-                 iyy="0.000498940" iyz="0.0"
-                 izz="0.003879257" />
+        <inertia ixx="0.003881243" ixy="0.0" ixz="0.0" iyy="0.000498940" iyz="0.0" izz="0.003879257" />
       </inertial>
     </link>
@@ -230,18 +325,18 @@
          files. However, for Gazebo simulation we need them, so we add them here.
          (Hence, don't publish them additionally!) -->
-	<joint name="camera_depth_joint" type="fixed">
-	  <origin xyz="0 ${2 * -kinect_cam_py} 0" rpy="0 0 0" />
-	  <parent link="camera_rgb_frame" />
-	  <child link="camera_depth_frame" />
-	</joint>
-	<link name="camera_depth_frame"/>
-	<joint name="camera_depth_optical_joint" type="fixed">
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
Commit message: kinect

File: src/vacumm_description/urdf/vacumm5.xacro (robot description, xacro)
@@ -2,5 +2,5 @@
 <robot xmlns:xacro="http://www.ros.org/wiki/xacro" name="vacumm_bot1">
   <xacro:property name="base_width" value="0.2"/>
-  <xacro:property name="base_len" value="0.16"/>
+  <xacro:property name="base_len" value="0.185"/>
   <xacro:property name="wheel_radius" value="0.04"/>
   <xacro:property name="base_wheel_gap" value="0.0175"/>
@@ -12,7 +12,7 @@
   <xacro:property name="caster_wheel_down_offset" value="0.0001"/>
   <xacro:property name="M_PI" value="3.1415926535897931" />
-  <xacro:property name="cam_px" value="0.025" />
-  <xacro:property name="cam_pz" value="${base_len-0.025}" />
-  <xacro:property name="kinect_cam_py" value="0"/>
+  <xacro:property name="cam_px" value="0.0" />
+  <xacro:property name="cam_pz" value="${base_len-0.0565}" />
+  <xacro:property name="kinect_cam_py" value="0.05"/>
   <xacro:property name="cam_or" value="0" />
   <xacro:property name="cam_op" value="0" />

Commit message: update

File: src/vacumm_description/urdf/vacumm5.xacro (robot description, xacro)
@@ -2,7 +2,7 @@
 <robot xmlns:xacro="http://www.ros.org/wiki/xacro" name="vacumm_bot1">
   <xacro:property name="base_width" value="0.2"/>
-  <xacro:property name="base_len" value="0.185"/>
-  <xacro:property name="wheel_radius" value="0.04"/>
-  <xacro:property name="base_wheel_gap" value="0.0175"/>
+  <xacro:property name="base_len" value="0.2"/>
+  <xacro:property name="wheel_radius" value="0.0425"/>
+  <xacro:property name="base_wheel_gap" value="0.0135"/>
   <xacro:property name="wheel_joint_offset" value="0"/>
   <xacro:property name="wheel_joint_drop_offset" value="-0.02"/>
