Commit message: update

File: src/vacumm_description/urdf/vacumm7.xacro (robot description, xacro)
@@ -241,4 +241,12 @@
     <child link="base_link" />
   </joint>
+  <link name="imu_link">
+  <origin xyz="0 0 0" rpy="0 0 0" />
+  </link>
+  <joint name="imu_link_joint" type="fixed">
+    <origin xyz="0 0 0" rpy="0 0 0" />
+    <parent link="base_link"/>
+    <child link="imu_link" />
+  </joint>
   <!-- <xacro:caster_wheel prefix="front" reflect="1"/> -->
   <xacro:caster_wheel prefix="back" reflect="-1"/>

Commit message: update

File: src/vacumm_description/urdf/vacumm7.xacro (robot description, xacro)
@@ -244,5 +244,5 @@
   <origin xyz="0 0 0" rpy="0 0 0" />
   </link>
-  <joint name="imu_link_joint" type="fixed">
+  <joint name="imu_link_joint" type="floating">
     <origin xyz="0 0 0" rpy="0 0 0" />
     <parent link="base_link"/>

Commit message: update

File: src/vacumm_description/urdf/vacumm7.xacro (robot description, xacro)
@@ -241,12 +241,4 @@
     <child link="base_link" />
   </joint>
-  <link name="imu_link">
-  <origin xyz="0 0 0" rpy="0 0 0" />
-  </link>
-  <joint name="imu_link_joint" type="floating">
-    <origin xyz="0 0 0" rpy="0 0 0" />
-    <parent link="base_link"/>
-    <child link="imu_link" />
-  </joint>
   <!-- <xacro:caster_wheel prefix="front" reflect="1"/> -->
   <xacro:caster_wheel prefix="back" reflect="-1"/>

Commit message: update4

File: src/vacumm_description/urdf/vacumm7.xacro (robot description, xacro)
@@ -1,9 +1,9 @@
 <?xml version="1.0"?>
 <robot xmlns:xacro="http://www.ros.org/wiki/xacro" name="vacumm_bot1">
-  <xacro:property name="base_width" value="0.191"/>
+  <xacro:property name="base_width" value="0.235"/>
   <xacro:property name="base_height" value="0.16"/>
   <xacro:property name="base_len" value="0.26"/>
   <xacro:property name="wheel_radius" value="0.04"/>
-  <xacro:property name="base_wheel_gap" value="0.01"/>
+  <xacro:property name="base_wheel_gap" value="0.0125"/>
   <xacro:property name="wheel_joint_offset" value="0.09"/>
   <xacro:property name="wheel_joint_drop_offset" value="-0.02"/>
